Commit message: updated xacro

File: inail_drill_urdf/urdf/inail_drill_macro.urdf.xacro (robot description, xacro)
@@ -9,6 +9,10 @@
   <xacro:property name="mm2m" value="1e-3" />
   <xacro:property name="sqmm2sqm" value="1e-6" />
-  <material name="drill_dark_grey"> <color rgba="0.1 0.1 0.1 1"/> </material>
-  <material name="drill_silver"> <color rgba="0.7 0.7 0.7 0.8"/> </material>
+  <material name="drill_dark_grey">
+    <color rgba="0.1 0.1 0.1 1"/>
+  </material>
+  <material name="drill_silver">
+    <color rgba="0.7 0.7 0.7 0.8"/>
+  </material>
     <!-- Drill Base Link -->
     <link name="drill_base">
@@ -40,6 +44,6 @@
         <geometry>
           <mesh filename="package://inail_drill_urdf/meshes/drill_chuck.stl" scale = "0.001 0.001 0.001"/>
-          <material name="drill_dark_grey"/>
         </geometry>
+        <material name="drill_dark_grey"/>
       </visual>
       <collision>

Commit message: updated drill on arm 2

File: inail_drill_urdf/urdf/inail_drill_macro.urdf.xacro (robot description, xacro)
@@ -10,8 +10,8 @@
   <xacro:property name="sqmm2sqm" value="1e-6" />
   <material name="drill_dark_grey">
-    <color rgba="0.1 0.1 0.1 1"/>
+    <color rgba="0.3 0.3 0.3 1"/>
   </material>
   <material name="drill_silver">
-    <color rgba="0.7 0.7 0.7 0.8"/>
+    <color rgba="0.6 0.6 0.7 1.0"/>
   </material>
     <!-- Drill Base Link -->
@@ -65,10 +65,10 @@
     </joint>
     <!-- Joint between drill base and drill chuck -->
-    <joint name="drill_joint" type="continuous">
+    <joint name="inail_drill_motor" type="continuous">
       <parent link="drill_base"/>
       <child link="drill_chuck"/>
       <origin xyz="0 0 ${188.5*mm2m}" rpy="0 0 0"/>
       <axis xyz="0 0 1"/>
-      <limit velocity="1000.0" effort="30.0"/>
+      <limit velocity="100.0" effort="30.0"/>
     </joint>
   </xacro:macro>
